File: Arduino 40hz audio and led.sch (EAGLE design)
At the start: 38 parts, among them IC1 LM7805, IC2 IRL-Z44N, IC3 LM741

Commit message: Should be final surface mount commit
This should be the final surface mount commit before making a new
version of the board with 'proper' through hole parts.
Connections:
- net N$14: now also U$4.P$1
- net N$15: now also U$6.P$1
- net N$6: now also U$3.P$1
Changed lines of the file:
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@@
 </variantdefs>
 <classes>
-<class number="0" name="default" width="0" drill="0">
+<class number="0" name="default" width="1.016" drill="0">
+<clearance class="0" value="0.508"/>
 </class>
-<class number="1" name="Thin20" width="0" drill="0">
+<class number="1" name="1mm" width="1.016" drill="0">
+<clearance class="1" value="0.508"/>
 </class>
-<class number="2" name="Medium25" width="0" drill="0">
+<class number="2" name="1.5mm" width="1.524" drill="0">
+<clearance class="2" value="0.508"/>
 </class>
-<class number="3" name="Medium30" width="0" drill="0">
+<class number="3" name="2mm" width="2.032" drill="0">
+<clearance class="3" value="0.508"/>
 </class>
 <class number="4" name="Large50" width="0" drill="0">
+<clearance class="4" value="0.508"/>
 </class>
 <class number="5" name="Large100" width="0" drill="0">
+<clearance class="5" value="0.508"/>
 </class>
 </classes>
@@
 </segment>
 </net>
-<net name="+12V" class="0">
+<net name="+12V" class="2">
 <segment>
 <pinref part="P+1" gate="1" pin="+12V"/>
@@
 </segment>
 </net>
-<net name="+5V" class="0">
+<net name="+5V" class="2">
 <segment>
 <pinref part="IC1" gate="G$1" pin="OUT"/>
@@
 <wire x1="58.42" y1="55.88" x2="58.42" y2="53.34" width="0.1524" layer="91"/>
 <wire x1="58.42" y1="53.34" x2="66.04" y2="53.34" width="0.1524" layer="91"/>
-<pinref part="U$7" gate="G$1" pin="P$1"/>
-<wire x1="73.66" y1="83.82" x2="66.04" y2="83.82" width="0.1524" layer="91"/>
-<junction x="66.04" y="83.82"/>
 <pinref part="JP3" gate="A" pin="2"/>
 <wire x1="68.58" y1="43.18" x2="68.58" y2="76.2" width="0.1524" layer="91"/>
 <wire x1="68.58" y1="76.2" x2="66.04" y2="76.2" width="0.1524" layer="91"/>
 <junction x="66.04" y="76.2"/>
+<pinref part="U$7" gate="G$1" pin="P$1"/>
+<wire x1="73.66" y1="83.82" x2="66.04" y2="83.82" width="0.1524" layer="91"/>
+<junction x="66.04" y="83.82"/>
 </segment>
 <segment>
@@
 </segment>
 </net>
-<net name="N$1" class="0">
+<net name="N$1" class="2">
 <segment>
 <pinref part="DUTY-CYCLE" gate="G$1" pin="S"/>
@@
 </segment>
 </net>
-<net name="N$2" class="0">
+<net name="N$2" class="2">
 <segment>
 <pinref part="U$1" gate="G$1" pin="D9"/>
@@
 </segment>
 </net>
-<net name="N$3" class="0">
+<net name="N$3" class="2">
 <segment>
 <pinref part="R1" gate="G$1" pin="1"/>
@@
 </segment>
 </net>
-<net name="N$4" class="0">
+<net name="N$4" class="2">
 <segment>
 <pinref part="R2" gate="G$1" pin="1"/>
@@
 </segment>
 </net>
-<net name="N$5" class="0">
+<net name="N$5" class="2">
 <segment>
 <pinref part="R3" gate="G$1" pin="1"/>
@@
 </segment>
 </net>
-<net name="N$13" class="0">
+<net name="N$13" class="2">
 <segment>
 <pinref part="IC3" gate="G$1" pin="6"/>
@@
 </segment>
 </net>
-<net name="N$14" class="0">
+<net name="N$14" class="2">
 <segment>
 <pinref part="U$1" gate="G$1" pin="A4"/>
 <wire x1="73.66" y1="50.8" x2="55.88" y2="50.8" width="0.1524" layer="91"/>
 <wire x1="55.88" y1="50.8" x2="55.88" y2="48.26" width="0.1524" layer="91"/>
-<wire x1="55.88" y1="48.26" x2="50.8" y2="48.26" width="0.1524" layer="91"/>
-</segment>
-</net>
-<net name="N$15" class="0">
-<segment>
-<wire x1="50.8" y1="35.56" x2="60.96" y2="35.56" width="0.1524" layer="91"/>
+<wire x1="55.88" y1="48.26" x2="48.26" y2="48.26" width="0.1524" layer="91"/>
+<pinref part="U$4" gate="G$1" pin="P$1"/>
+</segment>
+</net>
+<net name="N$15" class="2">
+<segment>
+<wire x1="48.26" y1="35.56" x2="60.96" y2="35.56" width="0.1524" layer="91"/>
 <wire x1="60.96" y1="35.56" x2="60.96" y2="48.26" width="0.1524" layer="91"/>
 <pinref part="U$1" gate="G$1" pin="A5"/>
 <wire x1="60.96" y1="48.26" x2="73.66" y2="48.26" width="0.1524" layer="91"/>
-</segment>
-</net>
-<net name="N$6" class="0">
+<pinref part="U$6" gate="G$1" pin="P$1"/>
+</segment>
+</net>
+<net name="N$6" class="2">
 <segment>
 <pinref part="C6" gate="G$1" pin="1"/>
 <wire x1="154.94" y1="50.8" x2="157.48" y2="50.8" width="0.1524" layer="91"/>
 <pinref part="R4" gate="G$1" pin="1"/>
-<wire x1="157.48" y1="50.8" x2="172.72" y2="50.8" width="0.1524" layer="91"/>
+<wire x1="157.48" y1="50.8" x2="175.26" y2="50.8" width="0.1524" layer="91"/>
 <wire x1="157.48" y1="48.26" x2="157.48" y2="50.8" width="0.1524" layer="91"/>
 <junction x="157.48" y="50.8"/>
-</segment>
-</net>
-<net name="N$8" class="0">
+<pinref part="U$3" gate="G$1" pin="P$1"/>
+</segment>
+</net>
+<net name="N$8" class="2">
 <segment>
 <pinref part="U$1" gate="G$1" pin="VIN"/>
@@
 </segment>
 </net>
-<net name="N$9" class="0">
+<net name="N$9" class="2">
 <segment>
 <pinref part="JP3" gate="A" pin="1"/>
@@
 </segment>
 </net>
-<net name="N$10" class="0">
+<net name="N$10" class="2">
 <segment>
 <pinref part="IC3" gate="G$1" pin="2"/>
@@
 </segment>
 </net>
-<net name="N$11" class="0">
+<net name="N$11" class="2">
 <segment>
 <pinref part="U$9" gate="G$1" pin="P$1"/>
@@
 </segment>
 </net>
-<net name="N$12" class="0">
+<net name="N$12" class="2">
 <segment>
 <pinref part="R6" gate="G$1" pin="2"/>
@@
 </sheet>
 </sheets>
+<errors>
+</errors>
 </schematic>
 </drawing>

Commit message: First commit after creating thruhole branch
This is the first commit after changing parts and the board for a
thru-hole design.
Parts:
- C1, C2: device jim_muppet_parts:CAP-POLARIZED-RADIAL-2.5MM-25V-20% -> SparkFun-Passives:CAP_POLPTH4
- C3, C4, C5, C6: device jim_muppet_parts:CAP-MEDIUM-MUPPET -> rcl:C-US050-025X075
- IC1, IC2: device jim_muppet_parts:V_REG_78XXSIDE -> SparkFun-PowerIC:V_REG_78XXSIDE
- R1, R2, R3, R4, R5, R6, R8: device jim_muppet_parts:RESISTORPTH-1/4W -> SparkFun-Passives:RESISTORPTH-1/4W
- R7: device jim_muppet_parts:RESISTORPTH-1/4W -> rcl:C-US050-025X075
Connections:
- net N$8: now also U$1.RAW; no longer U$1.VIN
Other:
- moved on the sheet: C3, C4, C5, C6

Commit message: First version of moving traces to the bottom.
First version of moving traces to the bottom.

Now to figure out how to mill this correctly, I'm guessing I need to
mirror it when I do the tools.  Anyway future Jim will judge how this
went.
Parts:
- removed U$7: PAD-2PIN-RECTANGLE, jim_muppet_parts:PAD-2PIN-RECTANGLE
- DUTY-CYCLE, VOLUME: device jim_muppet_parts:POTENTIOMETER -> jim_muppet_parts:POTENTIOMETERTHRUHOLE
- IC3: device jim_muppet_parts:DUAL-INLINE-8DIL08-2 -> jim_muppet_parts:DUAL-INLINE-8THRUHOLE8
- JP2, JP3: device jim_muppet_parts:JUMPER-JP1E -> jim_muppet_parts:JUMPER-JP1ETHRUHOLE
- P+1: value +12V -> (none); device jim_muppet_parts:+12V -> jim_muppet_parts:+12VTHRUHOLE
- P+2: value +5V -> (none); device jim_muppet_parts:+5V -> jim_muppet_parts:+5VTHRUHOLE
- P+3: value +6V -> (none); device jim_muppet_parts:+6V -> jim_muppet_parts:+6VTHRUHOLE
- U$1: value ARDUINO-NANO -> (none); device jim_muppet_parts:ARDUINO-NANO -> jim_muppet_parts:ARDUINO-NANOTHRUHOLE
- U$10, U$11, U$12, U$13: value DRILL-HOLE-4MM -> DRILL-HOLE-4MMTHRUHOLE; device jim_muppet_parts:DRILL-HOLE-4MM -> jim_muppet_parts:DRILL-HOLE-4MMTHRUHOLE
- U$14, U$4, U$6, U$9: device jim_muppet_parts:PAD-1PIN-RECTANGLE175 -> jim_muppet_parts:PAD-1PIN-RECTANGLETHRUHOLE175
- U$2, U$5, U$8: device jim_muppet_parts:PROBE-POINTPROBE_POINT_1 -> jim_muppet_parts:PROBE-POINTTHRUHOLE1
- U$3: device jim_muppet_parts:PAD-1PIN-RECTANGLE200 -> jim_muppet_parts:PAD-1PIN-RECTANGLETHRUHOLE175
Connections:
- net +5V: no longer U$7.P$1
- net N$8: now also U$1.VIN; no longer U$1.RAW
Other:
- moved on the sheet: R7
Changed lines of the file:
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@@
 <?xml version="1.0" encoding="utf-8"?>
 <!DOCTYPE eagle SYSTEM "eagle.dtd">
-<eagle version="9.4.2">
+<eagle version="9.2.2">
 <drawing>
 <settings>
@@
 </classes>
 <parts>
-<part name="U$1" library="jim_muppet_parts" deviceset="ARDUINO-NANO" device=""/>
+<part name="U$1" library="jim_muppet_parts" deviceset="ARDUINO-NANO" device="THRUHOLE"/>
 <part name="R1" library="SparkFun-Passives" deviceset="RESISTOR" device="PTH-1/4W" value="39k"/>
 <part name="R2" library="SparkFun-Passives" deviceset="RESISTOR" device="PTH-1/4W" value="39k"/>
@@
 <part name="IC1" library="SparkFun-PowerIC" deviceset="V_REG_78XX" device="SIDE" value="LM7805"/>
 <part name="IC2" library="SparkFun-PowerIC" deviceset="V_REG_78XX" device="SIDE" value="IRL-Z44N"/>
-<part name="P+1" library="jim_muppet_parts" deviceset="+12V" device=""/>
-<part name="IC3" library="jim_muppet_parts" deviceset="DUAL-INLINE-8" device="DIL08-2" value="LM741"/>
+<part name="P+1" library="jim_muppet_parts" deviceset="+12V" device="THRUHOLE"/>
+<part name="IC3" library="jim_muppet_parts" deviceset="DUAL-INLINE-8" device="THRUHOLE8" value="LM741"/>
 <part name="C1" library="SparkFun-Passives" deviceset="CAP_POL" device="PTH4" value="10uF"/>
 <part name="C2" library="SparkFun-Passives" deviceset="CAP_POL" device="PTH4" value="100uF"/>
@@
 <part name="SUPPLY3" library="supply2" library_urn="urn:adsk.eagle:library:372" deviceset="GND" device=""/>
 <part name="SUPPLY4" library="supply2" library_urn="urn:adsk.eagle:library:372" deviceset="GND" device=""/>
-<part name="P+2" library="jim_muppet_parts" deviceset="+5V" device=""/>
+<part name="P+2" library="jim_muppet_parts" deviceset="+5V" device="THRUHOLE"/>
 <part name="SUPPLY5" library="supply2" library_urn="urn:adsk.eagle:library:372" deviceset="GND" device=""/>
-<part name="DUTY-CYCLE" library="jim_muppet_parts" deviceset="POTENTIOMETER" device="" package3d_urn="urn:adsk.eagle:package:22726/1" value="10K"/>
-<part name="VOLUME" library="jim_muppet_parts" deviceset="POTENTIOMETER" device="" package3d_urn="urn:adsk.eagle:package:22726/1" value="100k"/>
+<part name="DUTY-CYCLE" library="jim_muppet_parts" deviceset="POTENTIOMETER" device="THRUHOLE" value="10K"/>
+<part name="VOLUME" library="jim_muppet_parts" deviceset="POTENTIOMETER" device="THRUHOLE" value="100k"/>
 <part name="SUPPLY6" library="supply2" library_urn="urn:adsk.eagle:library:372" deviceset="GND" device=""/>
 <part name="R7" library="rcl" library_urn="urn:adsk.eagle:library:334" deviceset="C-US" device="050-025X075" package3d_urn="urn:adsk.eagle:package:23637/1" value="600R"/>
-<part name="U$7" library="jim_muppet_parts" deviceset="PAD-2PIN-RECTANGLE" device=""/>
-<part name="U$5" library="jim_muppet_parts" deviceset="PROBE-POINT" device="PROBE_POINT_1" value="+/- 6v virt gnd"/>
-<part name="P+3" library="jim_muppet_parts" deviceset="+6V" device=""/>
-<part name="JP2" library="jim_muppet_parts" deviceset="JUMPER-JP1E" device="" package3d_urn="urn:adsk.eagle:package:15455/1"/>
-<part name="JP3" library="jim_muppet_parts" deviceset="JUMPER-JP1E" device="" package3d_urn="urn:adsk.eagle:package:15455/1"/>
+<part name="U$5" library="jim_muppet_parts" deviceset="PROBE-POINT" device="THRUHOLE1" value="+/- 6v virt gnd"/>
+<part name="P+3" library="jim_muppet_parts" deviceset="+6V" device="THRUHOLE"/>
+<part name="JP2" library="jim_muppet_parts" deviceset="JUMPER-JP1E" device="THRUHOLE"/>
+<part name="JP3" library="jim_muppet_parts" deviceset="JUMPER-JP1E" device="THRUHOLE"/>
 <part name="R8" library="SparkFun-Passives" deviceset="RESISTOR" device="PTH-1/4W" value="4k"/>
-<part name="U$3" library="jim_muppet_parts" deviceset="PAD-1PIN-RECTANGLE" device="200" value="SINE out"/>
-<part name="U$2" library="jim_muppet_parts" deviceset="PROBE-POINT" device="PROBE_POINT_1" value="-6v test point"/>
-<part name="U$8" library="jim_muppet_parts" deviceset="PROBE-POINT" device="PROBE_POINT_1" value="+6v test point"/>
-<part name="U$9" library="jim_muppet_parts" deviceset="PAD-1PIN-RECTANGLE" device="175" value="PAD-1PIN-RECTANGLE175"/>
-<part name="U$10" library="jim_muppet_parts" deviceset="DRILL-HOLE-4MM" device=""/>
-<part name="U$11" library="jim_muppet_parts" deviceset="DRILL-HOLE-4MM" device=""/>
-<part name="U$12" library="jim_muppet_parts" deviceset="DRILL-HOLE-4MM" device=""/>
-<part name="U$13" library="jim_muppet_parts" deviceset="DRILL-HOLE-4MM" device=""/>
-<part name="U$4" library="jim_muppet_parts" deviceset="PAD-1PIN-RECTANGLE" device="175" value="SCL"/>
-<part name="U$6" library="jim_muppet_parts" deviceset="PAD-1PIN-RECTANGLE" device="175" value="PAD-1PIN-RECTANGLE175"/>
-<part name="U$14" library="jim_muppet_parts" deviceset="PAD-1PIN-RECTANGLE" device="175" value="PAD-1PIN-RECTANGLE175"/>
+<part name="U$3" library="jim_muppet_parts" deviceset="PAD-1PIN-RECTANGLE" device="THRUHOLE175" value="SINE out"/>
+<part name="U$2" library="jim_muppet_parts" deviceset="PROBE-POINT" device="THRUHOLE1" value="-6v test point"/>
+<part name="U$8" library="jim_muppet_parts" deviceset="PROBE-POINT" device="THRUHOLE1" value="+6v test point"/>
+<part name="U$9" library="jim_muppet_parts" deviceset="PAD-1PIN-RECTANGLE" device="THRUHOLE175" value="PAD-1PIN-RECTANGLE175"/>
+<part name="U$10" library="jim_muppet_parts" deviceset="DRILL-HOLE-4MM" device="THRUHOLE" value="DRILL-HOLE-4MMTHRUHOLE"/>
+<part name="U$11" library="jim_muppet_parts" deviceset="DRILL-HOLE-4MM" device="THRUHOLE" value="DRILL-HOLE-4MMTHRUHOLE"/>
+<part name="U$12" library="jim_muppet_parts" deviceset="DRILL-HOLE-4MM" device="THRUHOLE" value="DRILL-HOLE-4MMTHRUHOLE"/>
+<part name="U$13" library="jim_muppet_parts" deviceset="DRILL-HOLE-4MM" device="THRUHOLE" value="DRILL-HOLE-4MMTHRUHOLE"/>
+<part name="U$4" library="jim_muppet_parts" deviceset="PAD-1PIN-RECTANGLE" device="THRUHOLE175" value="SCL"/>
+<part name="U$6" library="jim_muppet_parts" deviceset="PAD-1PIN-RECTANGLE" device="THRUHOLE175" value="PAD-1PIN-RECTANGLE175"/>
+<part name="U$14" library="jim_muppet_parts" deviceset="PAD-1PIN-RECTANGLE" device="THRUHOLE175" value="PAD-1PIN-RECTANGLE175"/>
 </parts>
 <sheets>
@@
 <attribute name="VALUE" x="144.145" y="36.195" size="1.778" layer="96" rot="R180"/>
 </instance>
-<instance part="R7" gate="G$1" x="119.38" y="22.86" smashed="yes" rot="R90">
-<attribute name="NAME" x="117.8814" y="19.05" size="1.778" layer="95" rot="R90"/>
-<attribute name="VALUE" x="122.682" y="19.05" size="1.778" layer="96" rot="R90"/>
-</instance>
-<instance part="U$7" gate="G$1" x="78.74" y="83.82" smashed="yes"/>
+<instance part="R7" gate="G$1" x="114.3" y="27.94" smashed="yes" rot="R180">
+<attribute name="NAME" x="118.11" y="26.4414" size="1.778" layer="95" rot="R180"/>
+<attribute name="VALUE" x="118.11" y="31.242" size="1.778" layer="96" rot="R180"/>
+</instance>
 <instance part="U$5" gate="G$1" x="20.32" y="0" smashed="yes" rot="R90">
 <attribute name="NAME" x="13.97" y="0" size="1.778" layer="95" rot="R180"/>
@@
 <pinref part="IC1" gate="G$1" pin="OUT"/>
 <wire x1="66.04" y1="53.34" x2="66.04" y2="76.2" width="0.1524" layer="91"/>
-<wire x1="66.04" y1="76.2" x2="66.04" y2="83.82" width="0.1524" layer="91"/>
-<wire x1="66.04" y1="83.82" x2="66.04" y2="96.52" width="0.1524" layer="91"/>
+<wire x1="66.04" y1="76.2" x2="66.04" y2="96.52" width="0.1524" layer="91"/>
 <wire x1="66.04" y1="96.52" x2="53.34" y2="96.52" width="0.1524" layer="91"/>
 <pinref part="P+2" gate="1" pin="+5V"/>
@@
 <wire x1="68.58" y1="76.2" x2="66.04" y2="76.2" width="0.1524" layer="91"/>
 <junction x="66.04" y="76.2"/>
-<pinref part="U$7" gate="G$1" pin="P$1"/>
-<wire x1="73.66" y1="83.82" x2="66.04" y2="83.82" width="0.1524" layer="91"/>
-<junction x="66.04" y="83.82"/>
 </segment>
 <segment>
@@
 <junction x="114.3" y="58.42"/>
 <wire x1="114.3" y1="58.42" x2="114.3" y2="45.72" width="0.1524" layer="91"/>
-<wire x1="114.3" y1="45.72" x2="114.3" y2="27.94" width="0.1524" layer="91"/>
-<wire x1="114.3" y1="27.94" x2="124.46" y2="22.86" width="0.1524" layer="91"/>
+<wire x1="114.3" y1="45.72" x2="114.3" y2="33.02" width="0.1524" layer="91"/>
 <pinref part="R7" gate="G$1" pin="2"/>
 <wire x1="124.46" y1="35.56" x2="124.46" y2="45.72" width="0.1524" layer="91"/>
@@
 <net name="N$8" class="2">
 <segment>
-<pinref part="U$1" gate="G$1" pin="RAW"/>
+<pinref part="U$1" gate="G$1" pin="VIN"/>
 <wire x1="73.66" y1="33.02" x2="66.04" y2="33.02" width="0.1524" layer="91"/>
 <wire x1="66.04" y1="33.02" x2="66.04" y2="25.4" width="0.1524" layer="91"/>
@@
 <junction x="119.38" y="15.24"/>
 <pinref part="R7" gate="G$1" pin="1"/>
-<wire x1="116.84" y1="22.86" x2="119.38" y2="15.24" width="0.1524" layer="91"/>
+<wire x1="114.3" y1="25.4" x2="119.38" y2="15.24" width="0.1524" layer="91"/>
 <wire x1="119.38" y1="15.24" x2="119.38" y2="12.7" width="0.1524" layer="91"/>
 <pinref part="R8" gate="G$1" pin="2"/>
